File: HW2/Board_ME433/me433mtc.brd (EAGLE design)
At the start: 50 x 50 mm, 22 parts, among them IC1 PIC32MX250F128B, IC2 MCP1702, J1 USBMINIB-MB-H, SW1 SLIDE, Y1 8MHz

Commit message: finished board
Parts:
- moved LED2 57.6 mm to (2.54, 8.89)
- moved LED1 56.6 mm to (44.5, 47.0)
- moved R1 53.0 mm to (48.3, 41.9)
- moved SW1 52.1 mm to (19.1, 48.3), turned to 180 degrees
- moved R2 51.3 mm to (6.35, 5.08), turned to 90 degrees
- moved J2 49.4 mm to (48.3, 12.7), turned to 270 degrees
- moved C2 20.4 mm to (20.3, 43.2), turned to 270 degrees
- moved C5 20.4 mm to (39.4, 43.2), turned to 270 degrees
- moved R3 6.84 mm to (39.4, 8.89), turned to 90 degrees
- moved R4 4.02 mm to (43.2, 15.2), turned to 180 degrees
- moved Y1 3.59 mm to (14.0, 17.8)
- moved C7 2.54 mm to (34.3, 17.8)
- moved C3 1.80 mm to (31.8, 35.6), turned to 0 degrees
- moved PB2 1.80 mm to (30.5, 2.54)
- moved PB1 1.80 mm to (39.4, 2.54)
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Connections:
- removed net N$16: C3.1, IC1.13
- net +3V3: now also C3.1, IC1.13
- net B4/USER: now also R3.1
- net MCLR: now also R4.1
Routing:
- net +3V3: track 0.00 -> 134.0 mm, vias 0 -> 2
- net +5V: track 0.00 -> 80.4 mm, vias 0 -> 4
- net MCLR: track 0.00 -> 67.4 mm, vias 0 -> 2
- net B4/USER: track 0.00 -> 55.8 mm
- net USBID: track 0.00 -> 55.7 mm, vias 0 -> 1
- net A4/LED: track 0.00 -> 49.9 mm, vias 0 -> 1
- net D-: track 0.00 -> 47.7 mm, vias 0 -> 2
- net PGD: track 0.00 -> 44.7 mm, vias 0 -> 1
- net PGC: track 0.00 -> 44.3 mm, vias 0 -> 1
- net D+: track 0.00 -> 39.5 mm
- net B9: track 0.00 -> 32.7 mm
- net B8: track 0.00 -> 32.3 mm
- net B7: track 0.00 -> 31.9 mm, vias 0 -> 1
- net B15: track 0.00 -> 23.1 mm
- net B14: track 0.00 -> 23.1 mm
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- added copper zone on layer 16, net GND

Commit message: Ready to be checked before order
Routing:
- net GND: track 12.6 -> 0.00 mm
- net D-: track 47.7 -> 46.2 mm
Other:
- board text added: "KILLAKILLA"
Changed lines of the file:
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@@
 <layer number="27" name="tValues" color="7" fill="1" visible="yes" active="yes"/>
 <layer number="28" name="bValues" color="7" fill="1" visible="yes" active="yes"/>
-<layer number="29" name="tStop" color="7" fill="3" visible="no" active="yes"/>
-<layer number="30" name="bStop" color="7" fill="6" visible="no" active="yes"/>
-<layer number="31" name="tCream" color="7" fill="4" visible="no" active="yes"/>
-<layer number="32" name="bCream" color="7" fill="5" visible="no" active="yes"/>
-<layer number="33" name="tFinish" color="6" fill="3" visible="no" active="yes"/>
-<layer number="34" name="bFinish" color="6" fill="6" visible="no" active="yes"/>
-<layer number="35" name="tGlue" color="7" fill="4" visible="no" active="yes"/>
-<layer number="36" name="bGlue" color="7" fill="5" visible="no" active="yes"/>
-<layer number="37" name="tTest" color="7" fill="1" visible="no" active="yes"/>
-<layer number="38" name="bTest" color="7" fill="1" visible="no" active="yes"/>
+<layer number="29" name="tStop" color="7" fill="3" visible="yes" active="yes"/>
+<layer number="30" name="bStop" color="7" fill="6" visible="yes" active="yes"/>
+<layer number="31" name="tCream" color="7" fill="4" visible="yes" active="yes"/>
+<layer number="32" name="bCream" color="7" fill="5" visible="yes" active="yes"/>
+<layer number="33" name="tFinish" color="6" fill="3" visible="yes" active="yes"/>
+<layer number="34" name="bFinish" color="6" fill="6" visible="yes" active="yes"/>
+<layer number="35" name="tGlue" color="7" fill="4" visible="yes" active="yes"/>
+<layer number="36" name="bGlue" color="7" fill="5" visible="yes" active="yes"/>
+<layer number="37" name="tTest" color="7" fill="1" visible="yes" active="yes"/>
+<layer number="38" name="bTest" color="7" fill="1" visible="yes" active="yes"/>
 <layer number="39" name="tKeepout" color="4" fill="11" visible="yes" active="yes"/>
 <layer number="40" name="bKeepout" color="1" fill="11" visible="yes" active="yes"/>
@@
 <layer number="42" name="bRestrict" color="1" fill="10" visible="yes" active="yes"/>
 <layer number="43" name="vRestrict" color="2" fill="10" visible="yes" active="yes"/>
-<layer number="44" name="Drills" color="7" fill="1" visible="no" active="yes"/>
-<layer number="45" name="Holes" color="7" fill="1" visible="no" active="yes"/>
-<layer number="46" name="Milling" color="3" fill="1" visible="no" active="yes"/>
-<layer number="47" name="Measures" color="7" fill="1" visible="no" active="yes"/>
+<layer number="44" name="Drills" color="7" fill="1" visible="yes" active="yes"/>
+<layer number="45" name="Holes" color="7" fill="1" visible="yes" active="yes"/>
+<layer number="46" name="Milling" color="3" fill="1" visible="yes" active="yes"/>
+<layer number="47" name="Measures" color="7" fill="1" visible="yes" active="yes"/>
 <layer number="48" name="Document" color="7" fill="1" visible="yes" active="yes"/>
 <layer number="49" name="Reference" color="7" fill="1" visible="yes" active="yes"/>
@@
 <wire x1="50" y1="50" x2="0" y2="50" width="0" layer="20"/>
 <wire x1="0" y1="50" x2="0" y2="0" width="0" layer="20"/>
-<dimension x1="2.54" y1="19.05" x2="-2.54" y2="19.05" x3="0" y3="12.7" textsize="1.778" layer="16"/>
+<text x="39.37" y="36.83" size="1.778" layer="22" rot="MR270">KILLAKILLA</text>
 </plain>
 <attributes>
@@
 </class>
 </classes>
-<designrules name="default">
+<designrules name="SeeedStudio_2layer_DRU_no_angle_20140221">
 <description language="de">&lt;b&gt;EAGLE Design Rules&lt;/b&gt;
 &lt;p&gt;
@@
 necessary adjustments and save your customized
 design rules under a new name.</description>
+<description language="zh">&lt;b&gt;Seeed Studio EAGLE Design Rules&lt;/b&gt;
+</description>
 <param name="layerSetup" value="(1*16)"/>
-<param name="mtCopper" value="0.035mm 0.035mm 0.035mm 0.035mm 0.035mm 0.035mm 0.035mm 0.035mm 0.035mm 0.035mm 0.035mm 0.035mm 0.035mm 0.035mm 0.035mm 0.035mm"/>
-<param name="mtIsolate" value="1.5mm 0.15mm 0.2mm 0.15mm 0.2mm 0.15mm 0.2mm 0.15mm 0.2mm 0.15mm 0.2mm 0.15mm 0.2mm 0.15mm 0.2mm"/>
-<param name="mdWireWire" value="8mil"/>
-<param name="mdWirePad" value="8mil"/>
-<param name="mdWireVia" value="8mil"/>
-<param name="mdPadPad" value="8mil"/>
-<param name="mdPadVia" value="8mil"/>
-<param name="mdViaVia" value="8mil"/>
-<param name="mdSmdPad" value="8mil"/>
-<param name="mdSmdVia" value="8mil"/>
-<param name="mdSmdSmd" value="8mil"/>
+<param name="mtCopper" value="0.035mm 0.0175mm 0.035mm 0.035mm 0.035mm 0.035mm 0.035mm 0.035mm 0.035mm 0.035mm 0.035mm 0.035mm 0.035mm 0.035mm 0.0175mm 0.035mm"/>
+<param name="mtIsolate" value="1.5mm 1.1mm 0.2mm 0.15mm 0.2mm 0.15mm 0.2mm 0.15mm 0.2mm 0.15mm 0.2mm 0.15mm 0.2mm 0.15mm 0.2mm"/>
+<param name="mdWireWire" value="6mil"/>
+<param name="mdWirePad" value="6mil"/>
+<param name="mdWireVia" value="6mil"/>
+<param name="mdPadPad" value="6mil"/>
+<param name="mdPadVia" value="6mil"/>
+<param name="mdViaVia" value="6mil"/>
+<param name="mdSmdPad" value="0mil"/>
+<param name="mdSmdVia" value="0mil"/>
+<param name="mdSmdSmd" value="0mil"/>
 <param name="mdViaViaSameLayer" value="8mil"/>
 <param name="mnLayersViaInSmd" value="2"/>
-<param name="mdCopperDimension" value="40mil"/>
-<param name="mdDrill" value="8mil"/>
+<param name="mdCopperDimension" value="10mil"/>
+<param name="mdDrill" value="10mil"/>
 <param name="mdSmdStop" value="0mil"/>
-<param name="msWidth" value="10mil"/>
-<param name="msDrill" value="24mil"/>
-<param name="msMicroVia" value="9.99mm"/>
+<param name="msWidth" value="6mil"/>
+<param name="msDrill" value="12mil"/>
+<param name="msMicroVia" value="12mil"/>
 <param name="msBlindViaRatio" value="0.5"/>
 <param name="rvPadTop" value="0.25"/>
@@
 <param name="rlMinPadBottom" value="10mil"/>
 <param name="rlMaxPadBottom" value="20mil"/>
-<param name="rlMinViaOuter" value="8mil"/>
+<param name="rlMinViaOuter" value="6mil"/>
 <param name="rlMaxViaOuter" value="20mil"/>
-<param name="rlMinViaInner" value="8mil"/>
+<param name="rlMinViaInner" value="6mil"/>
 <param name="rlMaxViaInner" value="20mil"/>
 <param name="rlMinMicroViaOuter" value="4mil"/>
@@
 <param name="psTop" value="-1"/>
 <param name="psBottom" value="-1"/>
-<param name="psFirst" value="-1"/>
+<param name="psFirst" value="0"/>
 <param name="psElongationLong" value="100"/>
 <param name="psElongationOffset" value="100"/>
 <param name="mvStopFrame" value="1"/>
 <param name="mvCreamFrame" value="0"/>
-<param name="mlMinStopFrame" value="4mil"/>
-<param name="mlMaxStopFrame" value="4mil"/>
+<param name="mlMinStopFrame" value="2mil"/>
+<param name="mlMaxStopFrame" value="2mil"/>
 <param name="mlMinCreamFrame" value="0mil"/>
 <param name="mlMaxCreamFrame" value="0mil"/>
-<param name="mlViaStopLimit" value="0mil"/>
+<param name="mlViaStopLimit" value="100mil"/>
 <param name="srRoundness" value="0"/>
 <param name="srMinRoundness" value="0mil"/>
@@
 <param name="checkAngle" value="0"/>
 <param name="checkFont" value="1"/>
-<param name="checkRestrict" value="1"/>
+<param name="checkRestrict" value="0"/>
 <param name="useDiameter" value="13"/>
 <param name="maxErrors" value="50"/>
@@
 <contactref element="C7" pad="-"/>
 <contactref element="C2" pad="2"/>
-<wire x1="33.02" y1="35.56" x2="34.29" y2="34.29" width="0.4064" layer="16"/>
-<wire x1="34.29" y1="34.29" x2="34.29" y2="29.21" width="0.4064" layer="16"/>
-<wire x1="34.29" y1="29.21" x2="29.21" y2="26.67" width="0.4064" layer="16"/>
 <polygon width="0.4064" layer="16">
 <vertex x="-3.81" y="52.07"/>
@@
 <vertex x="-3.81" y="53.34"/>
 </polygon>
-<wire x1="44.45" y1="2.54" x2="35.56" y2="2.54" width="0" layer="19" extent="1-1"/>
+<wire x1="35.56" y1="2.54" x2="44.45" y2="2.54" width="0" layer="19" extent="1-1"/>
 </signal>
 <signal name="USBID">
@@
 <contactref element="J1" pad="D-"/>
 <contactref element="IC1" pad="22"/>
-<wire x1="7.71" y1="45.25" x2="3.81" y2="45.72" width="0.4064" layer="1"/>
-<via x="3.81" y="45.72" extent="1-16" drill="0.6"/>
-<wire x1="3.81" y1="45.72" x2="6.35" y2="43.18" width="0.4064" layer="16"/>
-<wire x1="6.35" y1="43.18" x2="6.35" y2="40.64" width="0.4064" layer="16"/>
+<wire x1="7.71" y1="45.25" x2="3.81" y2="44.45" width="0.4064" layer="1"/>
+<via x="3.81" y="44.45" extent="1-16" drill="0.6"/>
+<wire x1="3.81" y1="44.45" x2="6.35" y2="40.64" width="0.4064" layer="16"/>
 <wire x1="6.35" y1="40.64" x2="8.89" y2="38.1" width="0.4064" layer="16"/>
 <wire x1="8.89" y1="38.1" x2="24.13" y2="38.1" width="0.4064" layer="16"/>
@@
 <contactref element="IC1" pad="5"/>
 <wire x1="48.26" y1="2.54" x2="44.45" y2="6.35" width="0.4064" layer="1"/>
-<wire x1="44.45" y1="6.35" x2="34.29" y2="6.35" width="0.4064" layer="1"/>
-<via x="34.29" y="6.35" extent="1-16" drill="0.6"/>
-<wire x1="34.29" y1="6.35" x2="27.94" y2="11.43" width="0.4064" layer="16"/>
+<wire x1="44.45" y1="6.35" x2="33.3375" y2="6.985" width="0.4064" layer="1"/>
+<via x="33.3375" y="6.985" extent="1-16" drill="0.6"/>
+<wire x1="33.3375" y1="6.985" x2="27.94" y2="11.43" width="0.4064" layer="16"/>
 <wire x1="27.94" y1="11.43" x2="22.86" y2="11.43" width="0.4064" layer="16"/>
 <wire x1="22.86" y1="11.43" x2="21.59" y2="12.7" width="0.4064" layer="16"/>
@@
 <wire x1="26.67" y1="15.24" x2="31.75" y2="17.78" width="0.4064" layer="1"/>
 </signal>
-<signal name="N$8">
-<via x="3.81" y="45.72" extent="1-16" drill="0.6"/>
-</signal>
 </signals>
